File: pcb-demo/03_nor_or_gates/74x02/74x02.kicad_sch (KiCad schematic)
At the start: 0 parts

Commit message: PCBデモ回路生成機能実装 その５
流石に回路図自動生成は駄目そう
Parts:
- added U1: 74LS02, symbol 74xx:74LS02
Connections:
- new net IN_A: U1.2
- new net IN_B: U1.3
- new net OUT_Y: U1.1
- no-connect marks 0 -> 9
Other:
- note added: "Demo: 74x02 (4回路2入力NORゲート) IC: 74HC02N, SN74HC02N, HD74HC02F, TC74HC02AF, 74S02N, SN74F02N NOTE: unused gate inputs must be tied to VCC or GND in final design."
- note removed: "TODO: 74xxライブラリから 74x02 シンボルを配置し 上記ピン配置・配線要点に従って回路を完成させてください。 usage/03_nor_or_gates/74x02/ の一次資料確認チェックリストも参照。"
- note removed: "【データシート】 https://www.ti.com/lit/ds/symlink/sn74hc02.pdf"
- note removed: "【ピン配置】 1=1Y 2=1A 3=1B 4=2Y 5=2A 6=2B 7=GND 8=3A 9=3B 10=3Y 11=4A 12=4B 13=4Y 14=VCC"
- note removed: "【回路概要】74x02 基本動作デモ（1回路） 電源: +5V（ロジックファミリにより範囲が異なるため一次資料で確認） IC: 74HC02N, SN74HC02N, HD74HC02F, TC74HC02AF, 74S02N, SN74F02N"
- note removed: "【配線要点】 ・VCC/GND: ピン表で確認した電源ピンに接続。0.1µFをIC直近に配置。 ・入力: スイッチでH/Lを切り替え（フローティング禁止）。 ・出力: LED＋抵抗で観測（出力ドライブ能力は一次資料で確認）。"
