File: pcb-demo/05_flipflops_latches/74x109/74x109.kicad_sch (KiCad schematic)
At the start: 0 parts

Commit message: PCBデモ回路生成機能実装 その５
流石に回路図自動生成は駄目そう
Other:
- note added: "TODO: 74xxライブラリから 74x109 シンボルを配置し 上記ピン配置・配線要点に従って回路を完成させてください。 usage/05_flipflops_latches/74x109/ の一次資料確認チェックリストも参照。"
- note added: "【データシート】 https://www.ti.com/lit/ds/symlink/sn74hc109.pdf"
- note added: "【ピン配置】 (ピン情報なし — usage/05_flipflops_latches/74x109/ を参照)"
- note added: "【回路概要】74x109 フリップフロップ/ラッチ 基本動作デモ 電源: +5V（ロジックファミリにより範囲が異なるため一次資料で確認） IC: SN74HC109N, SN74F109N, SN74LS109AN, MC74F109N"
- note added: "【配線要点】 ・電源（VCC/GND）: ピン表で確認した電源ピンに接続。0.1µFのデカップリングコンデンサをIC VCC〜GND間の直近（できれば5mm以内）に配置。 ・入力のフローティング禁止: 未使用入力は必ずVCCまたはGNDに接続。CMOS系（74HC等）は特に重要（誤動作・貫通電流の原因）。 ・出力電流: LED駆動電流（目安8〜10mA）が出力定格以内であることを一次資料で確認。"
- note removed: "TODO: KiCadの標準ライブラリ (74xx) からシンボルを配置して回路を作成してください。 ピン配置・真理値表は usage/05_flipflops_latches/74x109/ の一次資料確認チェックリストを参照。"
Changed lines of the file:
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@@
   (title_block
     (title "74x109 Demo Circuit")
-    (date "2026-05-30")
+    (date "2026-06-15")
     (rev "0.1")
     (company "7400 Series Collection")
@@
     (comment 4 "IC: SN74HC109N, SN74F109N, SN74LS109AN, MC74F109N")
   )
-  (text "TODO: KiCadの標準ライブラリ (74xx) からシンボルを配置して回路を作成してください。\nピン配置・真理値表は usage/05_flipflops_latches/74x109/ の一次資料確認チェックリストを参照。"
-    (at 50 100 0)
-    (effects
-      (font
-        (size 1.5 1.5)
-      )
-    )
+  (text "【回路概要】74x109 フリップフロップ/ラッチ 基本動作デモ\n電源: +5V（ロジックファミリにより範囲が異なるため一次資料で確認）\nIC: SN74HC109N, SN74F109N, SN74LS109AN, MC74F109N"
+    (at 10 15 0)
+    (effects (font (size 1.5 1.5)))
+  )
+  (text "【ピン配置】\n(ピン情報なし — usage/05_flipflops_latches/74x109/ を参照)"
+    (at 10 38 0)
+    (effects (font (size 1.27 1.27)))
+  )
+  (text "【配線要点】\n・電源（VCC/GND）: ピン表で確認した電源ピンに接続。0.1µFのデカップリングコンデンサをIC VCC〜GND間の直近（できれば5mm以内）に配置。\n・入力のフローティング禁止: 未使用入力は必ずVCCまたはGNDに接続。CMOS系（74HC等）は特に重要（誤動作・貫通電流の原因）。\n・出力電流: LED駆動電流（目安8〜10mA）が出力定格以内であることを一次資料で確認。"
+    (at 10 68 0)
+    (effects (font (size 1.27 1.27)))
+  )
+  (text "【データシート】\nhttps://www.ti.com/lit/ds/symlink/sn74hc109.pdf"
+    (at 10 95 0)
+    (effects (font (size 1.27 1.27)))
+  )
+  (text "TODO: 74xxライブラリから 74x109 シンボルを配置し\n上記ピン配置・配線要点に従って回路を完成させてください。\nusage/05_flipflops_latches/74x109/ の一次資料確認チェックリストも参照。"
+    (at 10 140 0)
+    (effects (font (size 1.5 1.5)) (justify left))
   )
   (sheet_instances
