File: pcb-demo/_carrier/tiles/74x08/74x08_tile.kicad_pcb (KiCad board)
At the start: 2 copper layers, 50 x 50 mm, 78 parts, among them J1 5V_IN, SW1 MSS12C02LS-BB2.0, SW10 MSS12C02LS-BB2.0, SW11 MSS12C02LS-BB2.0, SW12 MSS12C02LS-BB2.0, SW13 MSS12C02LS-BB2.0, SW14 MSS12C02LS-BB2.0, SW15 MSS12C02LS-BB2.0, SW16 MSS12C02LS-BB2.0, SW17 MSS12C02LS-BB2.0, SW18 MSS12C02LS-BB2.0, SW19 MSS12C02LS-BB2.0, SW2 MSS12C02LS-BB2.0, SW3 MSS12C02LS-BB2.0, SW4 MSS12C02LS-BB2.0, SW5 MSS12C02LS-BB2.0, SW6 MSS12C02LS-BB2.0, SW8 MSS12C02LS-BB2.0, SW9 MSS12C02LS-BB2.0, U1 DIP20_Socket_300mil

Commit message: DRCレポート、ERCレポート、および混合パネル生成用のスクリプト追加
- 74x21タイルのDRCおよびERCレポートを作成（違反なし）
- スペシメンタイル用のフットプリントライブラリテーブルを追加
- 74x244タイル用のPNG画像追加
- スペシメンタイルの混合パネルを生成するスクリプト実装：2x2構成およびBOMの統合を可能に
- 既存のSpecimenタイル生成スクリプトに、CJKテキストの折り返し機能を追加
Other:
- board text added: "4回路2入力AND"
- board text added: "7400 Specimen Tile v0.1 74x08"
- board text added: "74x08"
- board text added: "AND gate"
- board text added: "ゲート"
- board text removed: "4回路2入力"
- board text removed: "7400 Specimen Tile v0.1 74x00"
- board text removed: "74x00"
- board text removed: "NAND gate"
- board text removed: "NANDゲート"

Commit message: DRC および ERC レポート、フットプリント・ライブラリ、およびドキュメントを追加
- 74x574タイルのDRCレポートを作成・違反事項と警告を特定。
- 回路図にエラーや警告がないことを示すERCレポートを生成。
- Specimen Tileのフットプリント用ライブラリテーブルを追加。
- Specimen Tile D27に関するセッション中の進捗状況と変更点についてドキュメント作成：シルクスクリーンの修正やフットプリントの問題への対応、タイルや混合パネルの生成コマンドについても言及
Parts:
- added MTG2: MountingHole_2.2mm_M2, MountingHole_2.2mm_M2, F.Cu at (46.5, 25.0)
Other:
- board text added: "4回路2入力ANDゲート"
- board text added: "Quad 2-input AND gate"
- board text removed: "4回路2入力AND"
- board text removed: "AND gate"
- board text removed: "Quad 2-input"
- board text removed: "ゲート"
