File: pcb-demo/_carrier/tiles/74x08/74x08_tile.kicad_sch (KiCad schematic)
At the start: 75 parts, among them J1 5V_IN, SW1 MSS12C02LS-BB2.0, SW10 MSS12C02LS-BB2.0, SW11 MSS12C02LS-BB2.0, SW12 MSS12C02LS-BB2.0, SW13 MSS12C02LS-BB2.0, SW14 MSS12C02LS-BB2.0, SW15 MSS12C02LS-BB2.0, SW16 MSS12C02LS-BB2.0, SW17 MSS12C02LS-BB2.0, SW18 MSS12C02LS-BB2.0, SW19 MSS12C02LS-BB2.0, SW2 MSS12C02LS-BB2.0, SW3 MSS12C02LS-BB2.0, SW4 MSS12C02LS-BB2.0, SW5 MSS12C02LS-BB2.0, SW6 MSS12C02LS-BB2.0, SW8 MSS12C02LS-BB2.0, SW9 MSS12C02LS-BB2.0, U1 DIP20_Socket_300mil

Commit message: DRCレポート、ERCレポート、および混合パネル生成用のスクリプト追加
- 74x21タイルのDRCおよびERCレポートを作成（違反なし）
- スペシメンタイル用のフットプリントライブラリテーブルを追加
- 74x244タイル用のPNG画像追加
- スペシメンタイルの混合パネルを生成するスクリプト実装：2x2構成およびBOMの統合を可能に
- 既存のSpecimenタイル生成スクリプトに、CJKテキストの折り返し機能を追加
Other:
- note added: "74x08 Specimen Tile v0.1 (Quad 2-input AND gate) DIP-14: VCC = contact 20, GND = contact 7 Cell k: SWk selects +5V/GND -> R(20+k) 220R -> contact k -> Rk 4.7k -> Dk -> GND Output contacts (per pinspec): SWk and R(20+k) are DNP, LED only (white; active_low = red + inverted) Clock contacts (attr=clock): tact SWTk + RCk/CKk RC + UGk 74LVC1G14 Schmitt trigger -> contact k Spec: pcb-demo/_carrier/READ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"
- note removed: "74x00 Specimen Tile v0.1 (Quad 2-input NAND gate) DIP-14: VCC = contact 20, GND = contact 7 Cell k: SWk selects +5V/GND -> R(20+k) 220R -> contact k -> Rk 4.7k -> Dk -> GND Output contacts (per pinspec): SWk and R(20+k) are DNP, LED only (white; active_low = red + inverted) Clock contacts (attr=clock): tact SWTk + RCk/CKk RC + UGk 74LVC1G14 Schmitt trigger -> contact k Spec: pcb-demo/_carrier/REA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"
- title: 74x00 Specimen Tile -> 74x08 Specimen Tile
